File: OLED64128Module_OEL1M4033FPC-A1-E/PCB_OLED_OEL1M4033FPC_A1_E/PCB_OLED_OEL1M4033FPC_A1_E.kicad_pcb (KiCad board)
At the start: 2 copper layers, 40 x 29 mm, 23 parts, among them J1 Conn_01x08_Male, J2 Conn_01x22_Female, SW1 SW_SPDT, U1 MT3608

Commit message: test OK.
Other:
- board text added: "2205"
- board text removed: "2204"
Changed lines of the file:
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@@
   (title_block
     (title "OLED_OEL1M4033FPC_A1")
-    (rev "0.9")
+    (date "2022-01-25")
+    (rev "1.0")
     (company "Lexsion.net")
   )
@@
   (gr_line (start 123.5 40) (end 123.5 55) (layer "F.SilkS") (width 0.15))
   (gr_line (start 95.5 40) (end 123.5 40) (layer "F.SilkS") (width 0.15))
-  (gr_circle (center 103.759 57.658) (end 104.14 57.658) (layer "B.Mask") (width 0) (fill solid))
+  (gr_circle (center 103.759 57.658) (end 104.179 57.658) (layer "B.Mask") (width 0) (fill solid))
   (gr_line (start 129.5 36) (end 129.5 59) (layer "Edge.Cuts") (width 0.1))
   (gr_arc (start 91 41) (mid 92.2947 41.6755) (end 93.5 42.5) (layer "Edge.Cuts") (width 0.1))
@@
     (effects (font (size 0.8 0.8) (thickness 0.12)) (justify mirror))
   )
-  (gr_text "2204" (at 97.663 60.071) (layer "B.SilkS")
+  (gr_text "2205" (at 97.663 60.071) (layer "B.SilkS")
     (effects (font (size 1 1) (thickness 0.15)) (justify mirror))
   )
