File: DAP_Link_CH55xT/PCB_DAP_Link_CH55xT/PCB_DAP_Link_CH55xT.kicad_pcb (KiCad board)
At the start: 2 copper layers, 41.1 x 21.3 mm, 44 parts, among them J1 USB_C_Receptacle_USB2.0, J2 JTAG+UART, Q1 8050, SW1 SW_Push, U1 SPX3819M5-L-3-3, U2 CH55xT, U3 SN74LVC1T45DBV, U4 SN74LVC1T45DBV

Commit message: Fix Silk for SW-GND&SW-RST at front.
Parts:
- moved kibuzzard-620E0A89 2.53 mm to (120.3, 66.0)
- moved kibuzzard-620E0A96 2.51 mm to (120.3, 68.5)
Changed lines of the file:
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@@
   (title_block
     (title "DAP_Link_CH55xT")
-    (rev "0.9")
+    (date "2022-02-25")
+    (rev "1.0")
     (company "lexsion.net")
+    (comment 1 "Fix Silk SW-GND&RST")
   )
   (layers
@@
   )
   (footprint "kibuzzard-620E0A96" (layer "F.Cu")
-    (at 120.284 65.97)
+    (at 120.3 68.48)
     (descr "Converted using: scripting")
     (tags "kb_params=7b27416c69676e6d656e7443686f696365273a20274c656674272c20274361704c65667443686f696365273a20275b272c2027436170526967687443686f696365273a20273e272c2027466f6e74436f6d626f426f78273a20275562756e74754d6f6e6f2d42272c20274865696768744374726c273a2027312e36272c20274d756c74694c696e6554657874273a2027525354272c202750616464696e67426f74746f6d4374726c273a202733272c202750616464696e674c6566744374726c273a202733272c202750616464696e6752696768744374726c273a202733272c202750616464696e67546f704374726c273a202733272c202757696474684374726c273a2027342e37277d")
@@
   )
   (footprint "kibuzzard-620E0A89" (layer "F.Cu")
-    (at 120.284 68.51)
+    (at 120.284 65.98)
     (descr "Converted using: scripting")
     (tags "kb_params=7b27416c69676e6d656e7443686f696365273a20274c656674272c20274361704c65667443686f696365273a20275b272c2027436170526967687443686f696365273a20273e272c2027466f6e74436f6d626f426f78273a20275562756e74754d6f6e6f2d42272c20274865696768744374726c273a2027312e36272c20274d756c74694c696e6554657874273a2027474e44272c202750616464696e67426f74746f6d4374726c273a202733272c202750616464696e674c6566744374726c273a202733272c202750616464696e6752696768744374726c273a202733272c202750616464696e67546f704374726c273a202733272c202757696474684374726c273a2027342e37277d")
